File: kicad/le_chiff_ble/le_chiff_ble.kicad_pcb (KiCad board)
At the start: 2 copper layers, 228.4 x 85 mm, 117 parts, among them J2 BL_CONN, Q1 AO3401A, SW1 ON_OFF, SW2 SW_RESET, SW3 Rotary_Encoder_Switch, U1 TP4056, U2 MS88SF2, U3 XC6206PxxxMR-Regulator_Linear, U4 DW01A, U5 FS8205, U6 USBLC6-2SC6

Commit message: change switch footprint to MX Hotswap. move diodes to top layer, so smd parts can be assembled by manufacturer
Parts:
- D10, D11, D12, D13, D14, D15, D16, D17, D18, D19, D20, D21, D22, D23, D24, D25, D26, D27, D28, D29, D30, D31, D32, D33, D34, D35, D36, D37, D4, D5, D6, D7, D8, D9: moved to F.Cu
- MX1, MX10, MX11, MX12, MX13, MX14, MX15, MX16, MX18, MX19, MX2, MX20, MX22, MX23, MX24, MX25, MX26, MX27, MX28, MX29, MX3, MX30, MX31, MX32, MX33, MX34, MX4, MX5, MX6, MX7, MX8, MX9: footprint Keebio-Parts:MX-Alps-Choc-1U-NoLED -> weteor:CherryMX_Hotswap
- MX17, MX21: footprint Keebio-Parts:MX-Alps-Choc-2U-StabFlip -> weteor:CherryMX_Hotswap
- moved D4 2.00 mm to (53.1, 77.1)
- moved D5 2.00 mm to (50.9, 96.0)
- moved D8 2.00 mm to (70.1, 93.5)
- moved D7 2.00 mm to (72.6, 74.7)
Routing:
- net vbus: track 225.1 -> 111.4 mm, vias 6 -> 5
- net Net-(D1-Pad1): track 112.7 -> 41.5 mm, vias 4 -> 2
- net Net-(D2-Pad1): track 90.0 -> 22.5 mm, vias 3 -> 2
- net col6: track 158.3 -> 118.5 mm, vias 3 -> 6
- net col7: track 165.2 -> 132.1 mm, vias 0 -> 3
- net col9: track 175.3 -> 153.7 mm, vias 0 -> 3
- net Net-(D6-Pad2): track 21.8 -> 7.91 mm, vias 0 -> 1
- net row0: track 247.1 -> 260.5 mm, vias 1 -> 10
- net Net-(D22-Pad2): track 16.6 -> 29.4 mm, vias 0 -> 1
- net Net-(D7-Pad2): track 25.2 -> 12.5 mm, vias 0 -> 1
- net Net-(D28-Pad2): track 10.4 -> 22.7 mm, vias 0 -> 1
- net col5: track 100.9 -> 88.8 mm, vias 0 -> 5
- net col8: track 157.0 -> 145.0 mm, vias 0 -> 3
- net Net-(D23-Pad2): track 14.5 -> 26.3 mm, vias 0 -> 1
- net Net-(D36-Pad2): track 11.6 -> 23.4 mm, vias 0 -> 1
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Other:
- net class Default removed
- net class Power removed
